File: Tube_amplifier.kicad_pcb (KiCad board)
At the start: 2 copper layers, 140 x 54 mm, 23 parts, among them J2 Input, J3 Conn_01x04, J4 output, T1 Transformer_SP_1S, U1 6N2P, U2 6P14P

Commit message: High Voltage stabilizer
Create high voltage stabilizer
Parts:
- added C3: 33n opt, spdf1626_lib:C_THT_K73-17_P7.00mm, F.Cu at (146.4, 107.2)
- added R12: 680R, spdf1626_lib:R_THT_025W, F.Cu at (151.3, 102.4)
- added R9: 220k opt, spdf1626_lib:R_THT_025W, F.Cu at (148.0, 102.4)
- moved R2 3.70 mm to (143.7, 101.4)
Connections:
- C12 pad 1: 240V -> Net-(C12-Pad1)
- U1 pad 6: 240V -> Net-(C12-Pad1)
Routing:
- net Net-(C3-Pad1): track 22.7 -> 73.4 mm
- net Net-(C12-Pad1): track 0.00 -> 17.9 mm
- net 240V: track 127.5 -> 115.8 mm
- net Net-(C8-Pad1): track 14.3 -> 20.3 mm
- net Net-(C3-Pad2): track 4.54 -> 9.84 mm
- net Net-(R2-Pad1): track 8.77 -> 5.07 mm
- removed copper zone on F.Cu, net GND
