File: Tube_amplifier.kicad_sch (KiCad schematic)
At the start: 99 parts, among them J2 Input, J3 Conn_01x04, J4 output, T1 Transformer_SP_1S, U1 6N2P, U2 6P14P

Commit message: Multiple PCB
Parts:
- removed C1, C2: 10uF, Capacitor_THT:CP_Radial_D5.0mm_P2.00mm, symbol Device:C
- removed C12, C13, C? (x3): 10uF, spdf1626_lib:C_THT_D10.0mm_P5.00mm, symbol Device:C
- removed C3: 33n opt, Capacitor_THT:C_Rect_L7.2mm_W3.0mm_P5.00mm_FKS2_FKP2_MKS2_MKP2, symbol Device:C
- removed C6: 1n, spdf1626_lib:C_THT_K73-17_P5.00mm, symbol Device:C
- removed C7, C9, C? (x5): 100n, spdf1626_lib:C_THT_K73-17_P9.00mm, symbol Device:C
- removed C8: 33n, Capacitor_THT:C_Rect_L7.2mm_W3.0mm_P5.00mm_FKS2_FKP2_MKS2_MKP2, symbol Device:C
- removed C? (x4): 6800pF, spdf1626_lib:C_THT_K73-17_P5.00mm, symbol Device:C
- removed C?: 100uF, Capacitor_THT:CP_Radial_D22.0mm_P10.00mm_SnapIn, symbol Device:C
- removed C?: 3300uF_10V, Capacitor_THT:CP_Radial_D6.3mm_P2.50mm, symbol Device:C
- removed D? (x7): 1n4007, Diode_THT:D_DO-41_SOD81_P12.70mm_Horizontal, symbol Device:D
- removed D? (x4): 1N5821, Diode_THT:D_DO-27_P15.24mm_Horizontal, symbol Device:D
- removed J2: Input, spdf1626_lib:PinHeader_1x02_P2.54mm, symbol Connector_Generic:Conn_01x02
- removed J3, J? (x4): Conn_01x04, spdf1626_lib:PinHeader_1x04_P2.54mm, symbol Connector_Generic:Conn_01x04
- removed J4, J? (x2): output, spdf1626_lib:PinHeader_1x02_P2.54mm, symbol Connector_Generic:Conn_01x02
- removed J? (x2): Conn_01x03, spdf1626_lib:PinHeader_1x03_P2.54mm, symbol Connector_Generic:Conn_01x03
- removed J?: Indication, spdf1626_lib:PinHeader_1x03_P2.54mm, symbol Connector_Generic:Conn_01x03
- removed J?: 220V, Connector_Phoenix_MC_HighVoltage:PhoenixContact_MCV_1,5_2-G-5.08_1x02_P5.08mm_Vertical, symbol Connector_Generic:Conn_01x02
- removed J?: HV_Transformer, spdf1626_lib:PinHeader_1x02_P2.54mm, symbol Connector_Generic:Conn_01x02
- removed J?: LV_Transformer, spdf1626_lib:PinHeader_1x02_P2.54mm, symbol Connector_Generic:Conn_01x02
- removed J?: Thyratrone, spdf1626_lib:PinHeader_1x03_P2.54mm, symbol Connector_Generic:Conn_01x03
- removed J?: Transformers, spdf1626_lib:PinHeader_1x02_P2.54mm, symbol Connector_Generic:Conn_01x02
- removed J?: AudioJack3, Connector_Audio:Jack_6.35mm_Neutrik_NMJ6HHD2_Horizontal, symbol Connector:AudioJack3
- removed J?: Anodes_enable, Connector_Phoenix_MC_HighVoltage:PhoenixContact_MCV_1,5_2-G-5.08_1x02_P5.08mm_Vertical, symbol Connector_Generic:Conn_01x02
- removed K?: SANYOU_SRD_Form_C, Relay_THT:Relay_SPDT_SANYOU_SRD_Series_Form_C, symbol Relay:SANYOU_SRD_Form_C
- removed L?: L_Coupled, spdf1626_lib:L_THT_PLA10, symbol spdf1626:L_Coupled
- removed NE?: Lamp_Neon, spdf1626_lib:PinHeader_1x02_P2.54mm, symbol Device:Lamp_Neon
- removed NE?: Anodes_OK, spdf1626_lib:PinHeader_1x02_P2.54mm, symbol Device:Lamp_Neon
- removed Q? (x4): MPSA42, Package_TO_SOT_THT:TO-92_Inline, symbol Transistor_BJT:MPSA42
- removed Q?: 2N3904, Package_TO_SOT_THT:TO-92_Inline, symbol Transistor_BJT:2N3904
- removed Q?: MJE13003, Package_TO_SOT_THT:TO-126-3_Vertical, symbol Transistor_BJT:MJE13003
- removed R1: 6k8, spdf1626_lib:R_THT_025W, symbol Device:R
- removed R12: 680R, spdf1626_lib:R_THT_025W, symbol Device:R
- removed R2: 220R*, spdf1626_lib:R_THT_1W, symbol Device:R
- removed R3, R5: 300k, spdf1626_lib:R_THT_025W, symbol Device:R
- removed R4, R8: 1k8, spdf1626_lib:R_THT_025W, symbol Device:R
- removed R6, R7: 200R, spdf1626_lib:R_THT_025W, symbol Device:R
- removed R9: 220k opt, spdf1626_lib:R_THT_025W, symbol Device:R
- removed R?: 40k, spdf1626_lib:R_THT_025W, symbol Device:R
- removed R?: 10k, spdf1626_lib:R_THT_025W, symbol Device:R
- removed R?: 50k, spdf1626_lib:R_THT_025W, symbol Device:R
- removed R? (x7): 1M, spdf1626_lib:R_THT_025W, symbol Device:R
- removed R?: 13k, spdf1626_lib:R_THT_025W, symbol Device:R
- removed R? (x2): 100k, spdf1626_lib:R_THT_025W, symbol Device:R
- removed R?: 100R, spdf1626_lib:R_THT_1W, symbol Device:R
- removed R?: 600R, spdf1626_lib:R_THT_025W, symbol Device:R
- removed RV1: 100k, spdf1626_lib:Potentiometer_THT_CA9V, symbol Device:R_Potentiometer
- removed RV? (x2): 470k, spdf1626_lib:Potentiometer_THT_CA9V, symbol Device:R_Potentiometer
- removed RV?: R_Potentiometer_Dual, Potentiometer_THT:Potentiometer_Alps_RK163_Dual_Horizontal, symbol Device:R_Potentiometer_Dual
- removed RV?: 10k, spdf1626_lib:Potentiometer_THT_CA9V, symbol Device:R_Potentiometer
- removed T1: Transformer_SP_1S, spdf1626_lib:Output_transformer, symbol Device:Transformer_SP_1S
- removed U1: 6N2P, spdf1626_lib:9-pin_tube_socket, symbol spdf1626:6N2P
- removed U2: 6P14P, spdf1626_lib:9-pin_tube_socket, symbol spdf1626:6P14P
- removed U?: SG2P, spdf1626_lib:7-pin_tube_socket, symbol spdf1626:SG2P
- removed U? (x2): 6E1P, spdf1626_lib:9-pin_tube_socket, symbol spdf1626:6E1P
Other:
- added sheet Amplifier (Amplifier.kicad_sch)
- added sheet Back_connectors (Back_connectors.kicad_sch)
- added sheet Front_connectors (Front_connectors.kicad_sch)
- added sheet Indication_board (Indication_board.kicad_sch)
- added sheet Power_supply (Power_supply.kicad_sch)
- note removed: "220V"
- note removed: "240V"
- note removed: "6V"
