File: Indication_board.kicad_sch (KiCad schematic)
At the start: 16 parts

Commit message: New power supply
Parts:
- gave numbers to parts that had none: 16
Changed lines of the file:
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@@
   (symbol (lib_id "power:GND") (at 116.84 80.01 0) (unit 1)
     (in_bom yes) (on_board yes) (fields_autoplaced)
-    (property "Reference" "#PWR?" (id 0) (at 116.84 86.36 0)
+    (property "Reference" "#PWR020" (id 0) (at 116.84 86.36 0)
       (effects (font (size 1.27 1.27)) hide)
     )
@@
   (symbol (lib_id "Device:R") (at 97.79 66.04 90) (unit 1)
     (in_bom yes) (on_board yes) (fields_autoplaced)
-    (property "Reference" "R?" (id 0) (at 97.79 59.69 90))
+    (property "Reference" "R11" (id 0) (at 97.79 59.69 90))
     (property "Value" "1M" (id 1) (at 97.79 62.23 90))
     (property "Footprint" "spdf1626_lib:R_THT_025W" (id 2) (at 97.79 67.818 90)
@@
   (symbol (lib_id "Connector_Generic:Conn_01x04") (at 95.25 95.25 0) (unit 1)
     (in_bom yes) (on_board yes) (fields_autoplaced)
-    (property "Reference" "J?" (id 0) (at 97.79 95.2499 0)
+    (property "Reference" "J5" (id 0) (at 97.79 95.2499 0)
       (effects (font (size 1.27 1.27)) (justify left))
     )
@@
   (symbol (lib_id "power:+6V") (at 121.92 77.47 180) (unit 1)
     (in_bom yes) (on_board yes)
-    (property "Reference" "#PWR?" (id 0) (at 121.92 73.66 0)
+    (property "Reference" "#PWR024" (id 0) (at 121.92 73.66 0)
       (effects (font (size 1.27 1.27)) hide)
     )
@@
   (symbol (lib_id "Device:C") (at 74.93 57.15 90) (mirror x) (unit 1)
     (in_bom yes) (on_board yes)
-    (property "Reference" "C?" (id 0) (at 73.66 50.8 90))
+    (property "Reference" "C11" (id 0) (at 73.66 50.8 90))
     (property "Value" "6800pF" (id 1) (at 73.66 53.34 90))
     (property "Footprint" "spdf1626_lib:C_THT_K73-17_P5.00mm" (id 2) (at 78.74 58.1152 0)
@@
   (symbol (lib_id "Device:R") (at 97.79 124.46 90) (unit 1)
     (in_bom yes) (on_board yes) (fields_autoplaced)
-    (property "Reference" "R?" (id 0) (at 97.79 118.11 90))
+    (property "Reference" "R12" (id 0) (at 97.79 118.11 90))
     (property "Value" "1M" (id 1) (at 97.79 120.65 90))
     (property "Footprint" "spdf1626_lib:R_THT_025W" (id 2) (at 97.79 126.238 90)
@@
   (symbol (lib_id "Connector_Generic:Conn_01x03") (at 59.69 59.69 0) (mirror y) (unit 1)
     (in_bom yes) (on_board yes) (fields_autoplaced)
-    (property "Reference" "J?" (id 0) (at 59.69 50.8 0))
+    (property "Reference" "J4" (id 0) (at 59.69 50.8 0))
     (property "Value" "Indication" (id 1) (at 59.69 53.34 0))
     (property "Footprint" "spdf1626_lib:PinHeader_1x03_P2.54mm" (id 2) (at 59.69 59.69 0)
@@
   (symbol (lib_id "spdf1626:6E1P") (at 119.38 123.19 0) (unit 1)
     (in_bom yes) (on_board yes) (fields_autoplaced)
-    (property "Reference" "U?" (id 0) (at 125.73 121.2849 0)
+    (property "Reference" "U5" (id 0) (at 125.73 121.2849 0)
       (effects (font (size 1.27 1.27)) (justify left))
     )
@@
   (symbol (lib_id "Device:C") (at 74.93 115.57 90) (unit 1)
     (in_bom yes) (on_board yes)
-    (property "Reference" "C?" (id 0) (at 73.66 121.92 90))
+    (property "Reference" "C12" (id 0) (at 73.66 121.92 90))
     (property "Value" "6800pF" (id 1) (at 73.66 119.38 90))
     (property "Footprint" "spdf1626_lib:C_THT_K73-17_P5.00mm" (id 2) (at 78.74 114.6048 0)
@@
   (symbol (lib_id "power:GND") (at 85.09 104.14 0) (unit 1)
     (in_bom yes) (on_board yes) (fields_autoplaced)
-    (property "Reference" "#PWR?" (id 0) (at 85.09 110.49 0)
+    (property "Reference" "#PWR019" (id 0) (at 85.09 110.49 0)
       (effects (font (size 1.27 1.27)) hide)
     )
@@
   (symbol (lib_id "Device:D") (at 91.44 132.08 90) (unit 1)
     (in_bom yes) (on_board yes)
-    (property "Reference" "D?" (id 0) (at 88.9 132.08 0))
+    (property "Reference" "D2" (id 0) (at 88.9 132.08 0))
     (property "Value" "1n4007" (id 1) (at 87.63 132.08 0)
       (effects (font (size 1.27 1.27)) hide)
@@
   (symbol (lib_id "power:GND") (at 116.84 138.43 0) (unit 1)
     (in_bom yes) (on_board yes) (fields_autoplaced)
-    (property "Reference" "#PWR?" (id 0) (at 116.84 144.78 0)
+    (property "Reference" "#PWR023" (id 0) (at 116.84 144.78 0)
       (effects (font (size 1.27 1.27)) hide)
     )
@@
   (symbol (lib_id "Device:R_Potentiometer") (at 85.09 124.46 0) (mirror x) (unit 1)
     (in_bom yes) (on_board yes) (fields_autoplaced)
-    (property "Reference" "RV?" (id 0) (at 82.55 123.1899 0)
+    (property "Reference" "RV4" (id 0) (at 82.55 123.1899 0)
       (effects (font (size 1.27 1.27)) (justify right))
     )
@@
   (symbol (lib_id "Device:R") (at 116.84 104.14 0) (mirror y) (unit 1)
     (in_bom yes) (on_board yes)
-    (property "Reference" "R?" (id 0) (at 110.49 102.87 0)
+    (property "Reference" "R14" (id 0) (at 110.49 102.87 0)
       (effects (font (size 1.27 1.27)) (justify right))
     )
@@
   (symbol (lib_id "Device:D") (at 91.44 73.66 90) (unit 1)
     (in_bom yes) (on_board yes)
-    (property "Reference" "D?" (id 0) (at 88.9 73.66 0))
+    (property "Reference" "D1" (id 0) (at 88.9 73.66 0))
     (property "Value" "1n4007" (id 1) (at 87.63 73.66 0)
       (effects (font (size 1.27 1.27)) hide)
@@
   (symbol (lib_id "power:GND") (at 69.85 72.39 0) (unit 1)
     (in_bom yes) (on_board yes) (fields_autoplaced)
-    (property "Reference" "#PWR?" (id 0) (at 69.85 78.74 0)
+    (property "Reference" "#PWR017" (id 0) (at 69.85 78.74 0)
       (effects (font (size 1.27 1.27)) hide)
     )
@@
   (symbol (lib_id "spdf1626:6E1P") (at 119.38 64.77 0) (unit 1)
     (in_bom yes) (on_board yes) (fields_autoplaced)
-    (property "Reference" "U?" (id 0) (at 125.73 62.8649 0)
+    (property "Reference" "U3" (id 0) (at 125.73 62.8649 0)
       (effects (font (size 1.27 1.27)) (justify left))
     )
@@
   (symbol (lib_id "Device:C") (at 104.14 73.66 0) (mirror y) (unit 1)
     (in_bom yes) (on_board yes)
-    (property "Reference" "C?" (id 0) (at 100.33 72.3899 0)
+    (property "Reference" "C13" (id 0) (at 100.33 72.3899 0)
       (effects (font (size 1.27 1.27)) (justify left))
     )
@@
   (symbol (lib_id "power:+6V") (at 81.28 91.44 0) (unit 1)
     (in_bom yes) (on_board yes) (fields_autoplaced)
-    (property "Reference" "#PWR?" (id 0) (at 81.28 95.25 0)
+    (property "Reference" "#PWR018" (id 0) (at 81.28 95.25 0)
       (effects (font (size 1.27 1.27)) hide)
     )
@@
   (symbol (lib_id "Device:R_Potentiometer") (at 85.09 66.04 0) (unit 1)
     (in_bom yes) (on_board yes) (fields_autoplaced)
-    (property "Reference" "RV?" (id 0) (at 82.55 64.7699 0)
+    (property "Reference" "RV2" (id 0) (at 82.55 64.7699 0)
       (effects (font (size 1.27 1.27)) (justify right))
     )
@@
   (symbol (lib_id "Device:C") (at 104.14 132.08 0) (mirror y) (unit 1)
     (in_bom yes) (on_board yes)
-    (property "Reference" "C?" (id 0) (at 100.33 130.8099 0)
+    (property "Reference" "C14" (id 0) (at 100.33 130.8099 0)
       (effects (font (size 1.27 1.27)) (justify left))
     )
@@
   (symbol (lib_id "Device:R") (at 116.84 45.72 0) (mirror y) (unit 1)
     (in_bom yes) (on_board yes)
-    (property "Reference" "R?" (id 0) (at 110.49 44.45 0)
+    (property "Reference" "R13" (id 0) (at 110.49 44.45 0)
       (effects (font (size 1.27 1.27)) (justify right))
     )
@@
   (symbol (lib_id "power:+6V") (at 121.92 135.89 180) (unit 1)
     (in_bom yes) (on_board yes)
-    (property "Reference" "#PWR?" (id 0) (at 121.92 132.08 0)
-      (effects (font (size 1.27 1.27)) hide)
-    )
+    (property "Reference" "#PWR025" (id 0) (at 121.92 132.08 0)
+      (effects (font (size 1.27 1.27)) hide)
+    )
